File: audio-esp32.kicad_pcb (KiCad board)
At the start: 2 copper layers, 37.1 x 24.4 mm, 24 parts, among them J1 Conn_01x03, U1 MSGEQ7, U2 MicrophoneModule, U3 USBCWrover

Commit message: update art
Parts:
- removed the G*** at (156.7, 79.2)
- removed the G*** at (153.2, 84.3)
- removed the G*** at (142.2, 88.1)
- removed the G*** at (132.3, 87.1)
- removed the G*** at (143.8, 71.9)
- removed the G*** at (145.8, 77.7)
- removed the G*** at (158.0, 87.6)
- removed the G*** at (151.1, 87.6)
- removed the G*** at (131.1, 75.2)
- removed the G*** at (133.9, 79.2)
- removed the G*** at (160.0, 69.6)
- removed the G*** at (142.5, 81.5)
- removed the G*** at (146.3, 85.6)
- added G***: LOGO, audio-esp32:FullArt, F.Cu at (144.3, 78.2)
- added G***: LOGO, LOGO, B.Cu at (132.8, 86.9)
Other:
- board text added: "JLCJLCJLCJLC"
