File: musikfoks.kicad_pcb (KiCad board)
At the start: 2 copper layers, 37.1 x 24.4 mm, 13 parts, among them J1 Conn_01x03, U1 MSGEQ7, U2 MicrophoneModule, U3 USBCWrover

Commit message: rename to musikfoks
Parts:
- G***: footprint audio-esp32:FullArt -> musikfoks:FullArt
- U2: footprint audio-esp32:MicrophoneModule -> musikfoks:MicrophoneModule
Changed lines of the file:
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@@
   (net 38 "LED_DATA")
   (net 39 "Net-(U3-Pad18)")
-  (module "audio-esp32:FullArt" (layer "F.Cu")
+  (module "musikfoks:FullArt" (layer "F.Cu")
     (at 144.272 78.232)
     (fp_text reference "G***" (at 0 0) (layer "F.SilkS") hide
@@
     )
   )
-  (module "audio-esp32:MicrophoneModule" (layer "F.Cu")
+  (module "musikfoks:MicrophoneModule" (layer "F.Cu")
     (at 149.86 90.17 180)
     (fp_text reference "U2" (at 0 -0.5 180 unlocked) (layer "F.SilkS") hide
