File: musikfoks.kicad_sch (KiCad schematic)
At the start: 10 parts, among them J1 Conn_01x03, U1 MSGEQ7, U2 MicrophoneModule, U3 USBCWrover

Commit message: rename to musikfoks
Parts:
- U2: footprint audio-esp32:MicrophoneModule -> musikfoks:MicrophoneModule; symbol audio-esp32:MicrophoneModule -> musikfoks:MicrophoneModule
Changed lines of the file:
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@@
     )
   )
-  (symbol (lib_id "audio-esp32:MicrophoneModule") (at 99.06 50.8 0) (unit 1)
+  (symbol (lib_id "musikfoks:MicrophoneModule") (at 99.06 50.8 0) (unit 1)
     (in_bom yes) (on_board yes)
     (property "Reference" "U2" (id 0) (at 90.17 49.53 0)
@@
       (effects (font (size 1.27 1.27)) (justify right))
     )
-    (property "Footprint" "audio-esp32:MicrophoneModule" (id 2) (at 99.06 50.8 0)
+    (property "Footprint" "musikfoks:MicrophoneModule" (id 2) (at 99.06 50.8 0)
       (effects (font (size 1.27 1.27)) hide)
     )
